File: right/right.sch (KiCad schematic (older format))
At the start: 85 parts

Commit message: key layout done
Parts:
- removed D? (x7): DIODE, symbol DIODE
- removed SW? (x7): SWITCH_PUSH, symbol SWITCH_PUSH
- added D12, D13, D14: DIODE, symbol DIODE
- added D7, D8, D9: LED, symbol LED
- added R1, R2, R3: RESISTOR, symbol RESISTOR
- added SW10: J, symbol SWITCH_PUSH
- added SW11: M, symbol SWITCH_PUSH
- added SW9: U, symbol SWITCH_PUSH
- SW1: renamed from SW?; value SWITCH_PUSH -> F7
- SW12: renamed from SW?; value SWITCH_PUSH -> F9
- SW13: renamed from SW?; value SWITCH_PUSH -> 9
- SW14: renamed from SW?; value SWITCH_PUSH -> I
- SW15: renamed from SW?; value SWITCH_PUSH -> K
- SW16: renamed from SW?; value SWITCH_PUSH -> ,
- SW17: renamed from SW?; value SWITCH_PUSH -> F10
- SW18: renamed from SW?; value SWITCH_PUSH -> 0
- SW19: renamed from SW?; value SWITCH_PUSH -> O
- SW2: renamed from SW?; value SWITCH_PUSH -> 7
- SW20: renamed from SW?; value SWITCH_PUSH -> L
- SW21: renamed from SW?; value SWITCH_PUSH -> .
- SW22: renamed from SW?; value SWITCH_PUSH -> RALT
- SW23: renamed from SW?; value SWITCH_PUSH -> F11
- SW24: renamed from SW?; value SWITCH_PUSH -> -
- SW25: renamed from SW?; value SWITCH_PUSH -> P
- SW26: renamed from SW?; value SWITCH_PUSH -> ;
- SW27: renamed from SW?; value SWITCH_PUSH -> /
- SW28: renamed from SW?; value SWITCH_PUSH -> RMETA
- SW29: renamed from SW?; value SWITCH_PUSH -> F12
- SW3: renamed from SW?; value SWITCH_PUSH -> Y
- SW30: renamed from SW?; value SWITCH_PUSH -> =
- SW31: renamed from SW?; value SWITCH_PUSH -> [
- SW32: renamed from SW?; value SWITCH_PUSH -> '
- SW33: renamed from SW?; value SWITCH_PUSH -> RCTL
- SW34: renamed from SW?; value SWITCH_PUSH -> BSPC
- SW35: renamed from SW?; value SWITCH_PUSH -> BSLSH
- SW36: renamed from SW?; value SWITCH_PUSH -> ]
- SW37: renamed from SW?; value SWITCH_PUSH -> ENTR
- SW38: renamed from SW?; value SWITCH_PUSH -> RSHIFT
- SW4: renamed from SW?; value SWITCH_PUSH -> H
- SW5: renamed from SW?; value SWITCH_PUSH -> N
- SW6: renamed from SW?; value SWITCH_PUSH -> RSPC
- SW7: renamed from SW?; value SWITCH_PUSH -> F8
- SW8: renamed from SW?; value SWITCH_PUSH -> 8
- gave numbers to parts that had none: 36
Connections:
- net ROW5: now reaches SW1.1, SW12.1, SW17.1, SW23.1, SW29.1, SW34.1, SW7.1, U1.28 (PB0)
- net COL0: now reaches D1.2 (K), D2.2 (K), D3.2 (K), D4.2 (K), D5.2 (K), D6.2 (K), U1.8 (PB6)
- net ROW4: now reaches SW13.1, SW18.1, SW2.1, SW24.1, SW30.1, SW35.1, SW8.1, U1.27 (PB1)
- net ROW3: now reaches SW14.1, SW19.1, SW25.1, SW3.1, SW31.1, SW36.1, U1.26 (PB2)
- net ROW3: now also SW9.1
- net ROW2: now reaches SW15.1, SW20.1, SW26.1, SW32.1, SW37.1, SW4.1, U1.25 (PB3)
- net ROW1: now reaches SW16.1, SW21.1, SW27.1, SW38.1, SW5.1, U1.10 (PB4)
- net ROW1: now also SW11.1
- net ROW0: now reaches SW28.1, SW33.1, SW6.1, U1.9 (PB5)
- net ROW0: no longer SW22.1
- net COL1: now reaches D10.2 (K), D11.2 (K), U1.24 (PB7)
- net COL1: now also D12.2 (K), D13.2 (K), D14.2 (K); no longer D25.2 (K)
- net COL2: now reaches D15.2 (K), D16.2 (K), D17.2 (K), D18.2 (K), D19.2 (K), U1.19 (PC6)
- net COL2: no longer D31.2 (K)
- net COL3: now reaches D20.2 (K), D21.2 (K), D22.2 (K), D23.2 (K), D24.2 (K), U1.18 (PC7)
- net COL3: now also D25.2 (K); no longer D36.2 (K)
- net COL4: now reaches D26.2 (K), D27.2 (K), D28.2 (K), D29.2 (K), D30.2 (K), U1.23 (PD0)
- net COL4: now also D31.2 (K)
- net COL5: now reaches D32.2 (K), D33.2 (K), D34.2 (K), D35.2 (K), U1.22 (PD1)
- net COL5: now also D36.2 (K)
- net COL6: now reaches D37.2 (K), D38.2 (K), D39.2 (K), D40.2 (K), D41.2 (K), U1.21 (PD2)
- net Earth: now reaches U1.1 (GND)
- net Earth: now also U1.15 (GND), D7.1 (K), D8.1 (K), D9.1 (K)
- net LED2: now reaches U1.12 (PD6)
- net LED0: now reaches U1.13 (PD4)
- net LED0: now also R1.2
- net LED1: now reaches U1.17 (PD5)
- net LED1: now also R2.2
- new net: D12.1 (A), SW9.2
- new net: D7.2 (A), R1.1
- new net: D13.1 (A), SW10.2
- new net: D14.1 (A), SW11.2
- new net: D8.2 (A), R2.1
- new net: D9.2 (A), R3.1
- new net LED3: R3.2
- no-connect marks 1 -> 0
Other:
- moved on the sheet: D25, D31, D36, SW22, SW28, SW33
